Commit message: Working URDF model with realsense camera

File: couchmobile_description/urdf/couch_description.urdf (robot description, URDF)
Before this commit: robot googly_john, 4 links, 3 joints
Links:
- added link camera_color_optical_frame; visual box size=0.1 0.1 0.1
- added link camera_depth_optical_frame; visual box size=0.1 0.1 0.1
Joints:
- added joint pole_to_color: type fixed, parent pole, child camera_color_optical_frame, origin xyz=0 0 2.2 rpy=0 -1.57 0, axis 0 0 1
- added joint pole_to_depth: type fixed, parent pole, child camera_depth_optical_frame, origin xyz=0 0 2.2 rpy=1.57 3.14 1.57, axis 0 0 1
- joint pole_to_laser: type continuous -> fixed

Commit message: Created camera_link to link to realsense cameras

File: couchmobile_description/urdf/couch_description.urdf (robot description, URDF)
Before this commit: robot googly_john, 6 links, 5 joints
Links:
- removed link camera_depth_optical_frame
- added link camera_link; visual box size=0.1 0.1 0.1
Joints:
- joint pole_to_depth: child camera_depth_optical_frame -> camera_link

Commit message: Added hokuyo model + current progress on lidar in gazebo.

File: couchmobile_description/urdf/couch_description.urdf (robot description, URDF)
Before this commit: robot googly_john, 6 links, 5 joints
Links:
- link base_link: mass None -> 10
- link laser: mass None -> 1e-5; geometry collision box size=0.1 0.1 0.1; visual mesh filename=package://couchmobile_description/meshes/hokuyo.dae
- link seating: mass None -> 10

Commit message: Added IMU simulation to URDF model

File: couchmobile_description/urdf/couch_description.urdf (robot description, URDF)
Before this commit: robot googly_john, 6 links, 5 joints
Links:
- added link imu_link, mass 0.02; visual box size=0.2 0.1 0.002
Joints:
- added joint base_to_imu: type fixed, parent base_link, child imu_link, origin xyz=0 0 0 rpy=0 0 0, axis 0 0 0
