Commit message: Fixed wheel rotation.

File: couchmobile_description/urdf/couch_description.urdf.xacro (robot description, xacro)
@@ -1,4 +1,6 @@
 <?xml version="1.0" ?>
 <robot name="googly_john" xmlns:xacro="http://ros.org/wiki/xacro">
+<!-- CONSTS -->
+    <xacro:property name="PI" value="3.14159265359"/>
 <!-- ROBOT DIMENSIONS -->
 <!-- SIMULATION PROPERTIES -->

File: couchmobile_description/urdf/wheel.macro.xacro (robot description, xacro)
@@ -4,4 +4,5 @@
     <xacro:property name="wheel_l" value="0.0254"/>
     <xacro:property name="wheel_m" value="0.3"/>
+    <xacro:property name="PI" value="3.14159265359"/>
     <xacro:macro name="wheel" params="prefix parent *origin">
         <joint name="${parent}_to_${prefix}_wheel" type="fixed">
@@ -12,5 +13,5 @@
         <link name="${prefix}_wheel">
             <visual>
-                <xacro:insert_block name="origin"/>
+                <origin xyz="0 0 0" rpy="${PI/2} 0 0"/>
                 <geometry>
                     <cylinder radius="${wheel_r}" length="${wheel_l}"/>
@@ -19,5 +20,5 @@
             </visual>
             <collision>
-                <xacro:insert_block name="origin"/>
+                <origin xyz="0 0 0" rpy="${PI/2} 0 0"/>
                 <geometry>
                     <cylinder radius="${wheel_r}" length="${wheel_l}"/>
@@ -25,5 +26,5 @@
             </collision>
             <inertial>
-                <xacro:insert_block name="origin"/>
+                <origin xyz="0 0 0" rpy="${PI/2} 0 0"/>
                 <mass value="${wheel_m}"/>
                 <inertia

Commit message: Changed front and back wheels to be joined to middle wheel and added transmission.

File: couchmobile_description/urdf/couch_description.urdf.xacro (robot description, xacro)
@@ -4,6 +4,7 @@
     <xacro:property name="PI" value="3.14159265359"/>
 <!-- ROBOT DIMENSIONS -->
+    <xacro:property name="wheel_separation" value="0.60"/>
 <!-- SIMULATION PROPERTIES -->
-    <xacro:property name="controller_fps" value="41.67"/>
+    <xacro:property name="controller_fps" value="40"/>
     <material name="grey">
         <color rgba="0.5 0.5 0.5 1"/>
@@ -60,7 +61,28 @@
     </link>
     <xacro:include filename="$(find couchmobile_description)/urdf/wheel.macro.xacro"/>
+    <xacro:wheel prefix="RM" parent="base_link">
+        <origin xyz="0 ${wheel_separation/2} 0" rpy="0 0 0" />
+    </xacro:wheel>
+    <xacro:wheel prefix="RF" parent="RM_wheel">
+        <origin xyz="0.2 0 0" rpy="0 0 0" />
+    </xacro:wheel>
+    <xacro:wheel prefix="RB" parent="RM_wheel">
+        <origin xyz="-0.2 0 0" rpy="0 0 0" />
+    </xacro:wheel>
     <xacro:wheel prefix="LM" parent="base_link">
-        <origin xyz="0 0.5 0" rpy="0 0 0" />
-    </xacro:wheel>
+        <origin xyz="0 -${wheel_separation/2} 0" rpy="0 0 0" />
+    </xacro:wheel>
+    <xacro:wheel prefix="LF" parent="LM_wheel">
+        <origin xyz="0.2 0 0" rpy="0 0 0" />
+    </xacro:wheel>
+    <xacro:wheel prefix="LB" parent="LM_wheel">
+        <origin xyz="-0.2 0 0" rpy="0 0 0" />
+    </xacro:wheel>
+    <xacro:wheel_transmission prefix="LM" parent="base_link"/>
+    <xacro:wheel_transmission prefix="RM" parent="base_link"/>
+    <xacro:wheel_coupling parent="LM_wheel" child="LF_wheel"/>
+    <xacro:wheel_coupling parent="LM_wheel" child="LB_wheel"/>
+    <xacro:wheel_coupling parent="RM_wheel" child="RF_wheel"/>
+    <xacro:wheel_coupling parent="RM_wheel" child="RB_wheel"/>
     <joint name="seating_to_pole" type="fixed">
         <parent link="seating"/>
@@ -189,17 +211,26 @@
     </gazebo>
 <!-- DRIVE SIMULATION -->
+<!--
     <gazebo>
-        <plugin name="differential_drive_controller" filename="libgazebo_ros_diff_drive.so">
-            <alwaysOn>true</alwaysOn>
-            <updateRate>${controller_fps}</updateRate>
-            <leftJoint>base_link_left_wheel_joint</leftJoint>
-            <rightJoint>base_link_right_wheel_joint</rightJoint>
-            <wheelSeparation>0.65</wheelSeparation>
-            <wheelDiameter>0.152</wheelDiameter>
-            <torque>30</torque>
-            <commandTopic>cmd_vel</commandTopic>
-            <odometryTopic>odom</odometryTopic>
-            <odometryFrame>odom</odometryFrame>
+        <plugin name="gazebo_ros_control" filename="libgazebo_ros_control.so">
+            <robotNamespace>/</robotNamespace>
+            <controlPeriod>0.024</controlPeriod>
+        </plugin>
+    </gazebo>
+-->
+    <gazebo>
+        <plugin name="skid_steer_drive_controller" filename="libgazebo_ros_skid_steer_drive.so">
+            <updateRate>100</updateRate>
+            <robotNamespace>/</robotNamespace>
+            <leftFrontJoint>LF_wheel</leftFrontJoint>
+            <rightFrontJoint>RF_wheel</rightFrontJoint>
+            <leftRearJoint>LB_wheel</leftRearJoint>
+            <rightRearJoint>RB_wheel</rightRearJoint>
+            <wheelSeparation>${wheel_separation}</wheelSeparation>
+            <wheelDiameter>0.154</wheelDiameter>
             <robotBaseFrame>base_link</robotBaseFrame>
+            <torque>20</torque>
+            <topicName>cmd_vel</topicName>
+            <broadcastTF>true</broadcastTF>
         </plugin>
     </gazebo>

File: couchmobile_description/urdf/wheel.macro.xacro (robot description, xacro)
@@ -1,5 +1,5 @@
 <?xml version="1.0"?>
 <robot xmlns:xacro="http://ros.org/wiki/xacro">
-    <xacro:property name="wheel_r" value="0.152"/>
+    <xacro:property name="wheel_r" value="0.0716"/>
     <xacro:property name="wheel_l" value="0.0254"/>
     <xacro:property name="wheel_m" value="0.3"/>
@@ -35,3 +35,25 @@
         </link>
     </xacro:macro>
+    <xacro:macro name="wheel_transmission" params="prefix parent">
+        <transmission name="${prefix}_wheel_trans">
+            <type>transmission_interface/SimpleTransmission</type>
+            <actuator name="${prefix}_wheel_motor">
+                <mechanicalReduction>1</mechanicalReduction>
+            </actuator>
+            <joint name="${parent}_to_${prefix}_wheel">
+                <hardwareInterface>hardware_interface/VelocityJointInterface</hardwareInterface>
+            </joint>
+        </transmission>
+    </xacro:macro>
+    <xacro:macro name="wheel_coupling" params="parent child">
+        <transmission name="${parent}_to_${child}_trans">
+            <type>transmission_interface/SimpleTransmission</type>
+            <actuator name="${parent}_to_${child}_motor">
+                <mechanicalReduction>1</mechanicalReduction>
+            </actuator>
+            <joint name="${parent}_to_${child}">
+                <hardwareInterface>hardware_interface/VelocityJointInterface</hardwareInterface>
+            </joint>
+        </transmission>
+    </xacro:macro>
 </robot>

Commit message: Working gazebo motion model. Response is slow.

File: couchmobile_description/urdf/couch_description.urdf.xacro (robot description, xacro)
@@ -62,27 +62,27 @@
     <xacro:include filename="$(find couchmobile_description)/urdf/wheel.macro.xacro"/>
     <xacro:wheel prefix="RM" parent="base_link">
-        <origin xyz="0 ${wheel_separation/2} 0" rpy="0 0 0" />
-    </xacro:wheel>
-    <xacro:wheel prefix="RF" parent="RM_wheel">
-        <origin xyz="0.2 0 0" rpy="0 0 0" />
-    </xacro:wheel>
-    <xacro:wheel prefix="RB" parent="RM_wheel">
-        <origin xyz="-0.2 0 0" rpy="0 0 0" />
+        <origin xyz="0 ${wheel_separation/2} 0" rpy="0 0 ${PI/2}" />
+    </xacro:wheel>
+    <xacro:wheel prefix="RF" parent="base_link">
+        <origin xyz="0.2 ${wheel_separation/2} 0" rpy="0 0 ${PI/2}" />
+    </xacro:wheel>
+    <xacro:wheel prefix="RB" parent="base_link">
+        <origin xyz="-0.2 ${wheel_separation/2} 0" rpy="0 0 ${PI/2}" />
     </xacro:wheel>
     <xacro:wheel prefix="LM" parent="base_link">
-        <origin xyz="0 -${wheel_separation/2} 0" rpy="0 0 0" />
-    </xacro:wheel>
-    <xacro:wheel prefix="LF" parent="LM_wheel">
-        <origin xyz="0.2 0 0" rpy="0 0 0" />
-    </xacro:wheel>
-    <xacro:wheel prefix="LB" parent="LM_wheel">
-        <origin xyz="-0.2 0 0" rpy="0 0 0" />
+        <origin xyz="0 -${wheel_separation/2} 0" rpy="0 0 ${PI/2}" />
+    </xacro:wheel>
+    <xacro:wheel prefix="LF" parent="base_link">
+        <origin xyz="0.2 -${wheel_separation/2} 0" rpy="0 0 ${PI/2}" />
+    </xacro:wheel>
+    <xacro:wheel prefix="LB" parent="base_link">
+        <origin xyz="-0.2 -${wheel_separation/2} 0" rpy="0 0 ${PI/2}" />
     </xacro:wheel>
     <xacro:wheel_transmission prefix="LM" parent="base_link"/>
     <xacro:wheel_transmission prefix="RM" parent="base_link"/>
-    <xacro:wheel_coupling parent="LM_wheel" child="LF_wheel"/>
-    <xacro:wheel_coupling parent="LM_wheel" child="LB_wheel"/>
-    <xacro:wheel_coupling parent="RM_wheel" child="RF_wheel"/>
-    <xacro:wheel_coupling parent="RM_wheel" child="RB_wheel"/>
+    <xacro:wheel_coupling parent_wheel="LM_wheel" child_wheel="LF_wheel" parent="base_link"/>
+    <xacro:wheel_coupling parent_wheel="LM_wheel" child_wheel="LB_wheel" parent="base_link"/>
+    <xacro:wheel_coupling parent_wheel="RM_wheel" child_wheel="RF_wheel" parent="base_link"/>
+    <xacro:wheel_coupling parent_wheel="RM_wheel" child_wheel="RB_wheel" parent="base_link"/>
     <joint name="seating_to_pole" type="fixed">
         <parent link="seating"/>
@@ -211,26 +211,21 @@
     </gazebo>
 <!-- DRIVE SIMULATION -->
-<!--
     <gazebo>
         <plugin name="gazebo_ros_control" filename="libgazebo_ros_control.so">
-            <robotNamespace>/</robotNamespace>
-            <controlPeriod>0.024</controlPeriod>
         </plugin>
     </gazebo>
--->
     <gazebo>
-        <plugin name="skid_steer_drive_controller" filename="libgazebo_ros_skid_steer_drive.so">
-            <updateRate>100</updateRate>
-            <robotNamespace>/</robotNamespace>
-            <leftFrontJoint>LF_wheel</leftFrontJoint>
-            <rightFrontJoint>RF_wheel</rightFrontJoint>
-            <leftRearJoint>LB_wheel</leftRearJoint>
-            <rightRearJoint>RB_wheel</rightRearJoint>
-            <wheelSeparation>${wheel_separation}</wheelSeparation>
+        <plugin name="differential_drive_controller" filename="libgazebo_ros_diff_drive.so">
+            <alwaysOn>true</alwaysOn>
+            <updateRate>${controller_fps}</updateRate>
+            <leftJoint>base_link_to_LM_wheel</leftJoint>
+            <rightJoint>base_link_to_RM_wheel</rightJoint>
+            <wheelSeparation>0.60</wheelSeparation>
             <wheelDiameter>0.154</wheelDiameter>
+            <torque>50</torque>
+            <commandTopic>cmd_vel</commandTopic>
+            <odometryTopic>odom</odometryTopic>
+            <odometryFrame>odom</odometryFrame>
             <robotBaseFrame>base_link</robotBaseFrame>
-            <torque>20</torque>
-            <topicName>cmd_vel</topicName>
-            <broadcastTF>true</broadcastTF>
         </plugin>
     </gazebo>

File: couchmobile_description/urdf/wheel.macro.xacro (robot description, xacro)
@@ -6,5 +6,5 @@
     <xacro:property name="PI" value="3.14159265359"/>
     <xacro:macro name="wheel" params="prefix parent *origin">
-        <joint name="${parent}_to_${prefix}_wheel" type="fixed">
+        <joint name="${parent}_to_${prefix}_wheel" type="continuous">
             <parent link="${parent}"/>
             <child link="${prefix}_wheel"/>
@@ -13,5 +13,5 @@
         <link name="${prefix}_wheel">
             <visual>
-                <origin xyz="0 0 0" rpy="${PI/2} 0 0"/>
+                <origin xyz="0 0 0" rpy="0 ${PI/2} 0"/>
                 <geometry>
                     <cylinder radius="${wheel_r}" length="${wheel_l}"/>
@@ -20,5 +20,5 @@
             </visual>
             <collision>
-                <origin xyz="0 0 0" rpy="${PI/2} 0 0"/>
+                <origin xyz="0 0 0" rpy="0 ${PI/2} 0"/>
                 <geometry>
                     <cylinder radius="${wheel_r}" length="${wheel_l}"/>
@@ -26,5 +26,5 @@
             </collision>
             <inertial>
-                <origin xyz="0 0 0" rpy="${PI/2} 0 0"/>
+                <origin xyz="0 0 0" rpy="0 ${PI/2} 0"/>
                 <mass value="${wheel_m}"/>
                 <inertia
@@ -34,4 +34,13 @@
             </inertial>
         </link>
+        <gazebo reference="${prefix}_wheel">
+            <mu1 value = "200.0"/>
+            <mu2 value = "100.0"/>
+            <kp value="1000000.0" />
+            <kd value="1.0" />
+            <fdir1 value="1 0 0"/>
+            <material>Gazebo/Grey/</material>
+            <selfCollide>false</selfCollide>
+        </gazebo>
     </xacro:macro>
     <xacro:macro name="wheel_transmission" params="prefix parent">
@@ -46,11 +55,11 @@
         </transmission>
     </xacro:macro>
-    <xacro:macro name="wheel_coupling" params="parent child">
-        <transmission name="${parent}_to_${child}_trans">
+    <xacro:macro name="wheel_coupling" params="parent_wheel child_wheel parent">
+        <transmission name="${parent_wheel}_to_${child_wheel}_trans">
             <type>transmission_interface/SimpleTransmission</type>
-            <actuator name="${parent}_to_${child}_motor">
+            <actuator name="${parent_wheel}_to_${child_wheel}_motor">
                 <mechanicalReduction>1</mechanicalReduction>
             </actuator>
-            <joint name="${parent}_to_${child}">
+            <joint name="${parent}_to_${child_wheel}">
                 <hardwareInterface>hardware_interface/VelocityJointInterface</hardwareInterface>
             </joint>

Commit message: Working skid drive in gazebo. Ready to test navigation.

File: couchmobile_description/urdf/couch_description.urdf.xacro (robot description, xacro)
@@ -81,8 +81,8 @@
     <xacro:wheel_transmission prefix="LM" parent="base_link"/>
     <xacro:wheel_transmission prefix="RM" parent="base_link"/>
-    <xacro:wheel_coupling parent_wheel="LM_wheel" child_wheel="LF_wheel" parent="base_link"/>
-    <xacro:wheel_coupling parent_wheel="LM_wheel" child_wheel="LB_wheel" parent="base_link"/>
-    <xacro:wheel_coupling parent_wheel="RM_wheel" child_wheel="RF_wheel" parent="base_link"/>
-    <xacro:wheel_coupling parent_wheel="RM_wheel" child_wheel="RB_wheel" parent="base_link"/>
+    <xacro:wheel_transmission prefix="LF" parent="base_link"/>
+    <xacro:wheel_transmission prefix="RF" parent="base_link"/>
+    <xacro:wheel_transmission prefix="LB" parent="base_link"/>
+    <xacro:wheel_transmission prefix="RB" parent="base_link"/>
     <joint name="seating_to_pole" type="fixed">
         <parent link="seating"/>
@@ -219,14 +219,31 @@
             <alwaysOn>true</alwaysOn>
             <updateRate>${controller_fps}</updateRate>
-            <leftJoint>base_link_to_LM_wheel</leftJoint>
-            <rightJoint>base_link_to_RM_wheel</rightJoint>
+            <leftJoint>base_link_to_LM_wheel base_link_to_LF_wheel base_link_to_LB_wheel</leftJoint>
+            <rightJoint>base_link_to_RM_wheel base_link_to_RF_wheel base_link_to_RB_wheel</rightJoint>
             <wheelSeparation>0.60</wheelSeparation>
             <wheelDiameter>0.154</wheelDiameter>
-            <torque>50</torque>
+            <torque>20</torque>
             <commandTopic>cmd_vel</commandTopic>
-            <odometryTopic>odom</odometryTopic>
-            <odometryFrame>odom</odometryFrame>
+            <odometryTopic>odom_truth</odometryTopic>
+            <odometryFrame>odom_truth</odometryFrame>
             <robotBaseFrame>base_link</robotBaseFrame>
         </plugin>
     </gazebo>
+<!--
+    <gazebo>
+        <plugin name="skid_steer_drive_controller" filename="libgazebo_ros_skid_steer_drive.so">
+            <updateRate>100.0</updateRate>
+            <leftFrontJoint>LF_wheel</leftFrontJoint>
+            <rightFrontJoint>RF_wheel</rightFrontJoint>
+            <leftRearJoint>LB_wheel</leftRearJoint>
+            <rightRearJoint>RB_wheel</rightRearJoint>
+            <wheelSeparation>0.6</wheelSeparation>
+            <wheelDiameter>0.154</wheelDiameter>
+            <robotBaseFrame>base_link</robotBaseFrame>
+            <torque>20</torque>
+            <topicName>cmd_vel</topicName>
+            <broadcastTF>false</broadcastTF>
+        </plugin>
+    </gazebo>
+    -->
 </robot>

File: couchmobile_description/urdf/wheel.macro.xacro (robot description, xacro)
@@ -5,4 +5,5 @@
     <xacro:property name="wheel_m" value="0.3"/>
     <xacro:property name="PI" value="3.14159265359"/>
+    <xacro:property name="inertia_scale" value="10"/>
     <xacro:macro name="wheel" params="prefix parent *origin">
         <joint name="${parent}_to_${prefix}_wheel" type="continuous">
@@ -29,12 +30,12 @@
                 <mass value="${wheel_m}"/>
                 <inertia
-                    ixx="${1/2*wheel_m*wheel_r**2}" ixy="0.0" ixz="0.0"
-                    iyy="${1/12*wheel_m*(3*wheel_r**2+wheel_l**2)}" iyz="0.0"
-                    izz="${1/12*wheel_m*(3*wheel_r**2+wheel_l**2)}"/>
+                    ixx="${inertia_scale*1/2*wheel_m*wheel_r**2}" ixy="0.0" ixz="0.0"
+                    iyy="${inertia_scale*1/12*wheel_m*(3*wheel_r**2+wheel_l**2)}" iyz="0.0"
+                    izz="${inertia_scale*1/12*wheel_m*(3*wheel_r**2+wheel_l**2)}"/>
             </inertial>
         </link>
         <gazebo reference="${prefix}_wheel">
-            <mu1 value = "200.0"/>
-            <mu2 value = "100.0"/>
+            <mu1 value = "1.0"/>
+            <mu2 value = "0.2"/>
             <kp value="1000000.0" />
             <kd value="1.0" />

Commit message: Working couchmobile navigation in simulation

File: couchmobile_description/urdf/couch_description.urdf.xacro (robot description, xacro)
@@ -3,4 +3,5 @@
 <!-- CONSTS -->
     <xacro:property name="PI" value="3.14159265359"/>
+    <xacro:property name="deg_to_rad" value="${PI/180}"/>
 <!-- ROBOT DIMENSIONS -->
     <xacro:property name="wheel_separation" value="0.60"/>
@@ -163,9 +164,14 @@
 <!-- CAMERA DEFINITION -->
 <!-- CAMERA SIMULATION -->
+<!--
     <xacro:include filename="$(find couchmobile_description)/urdf/realsense-d435.macro.xacro"/>
-    <!-- Create camera instance -->
     <xacro:sensor-d435 prefix="" parent="pole">
         <origin xyz="0 0 2.2" rpy="0 0 0" />
     </xacro:sensor-d435>
+-->
+    <xacro:include filename="$(find realsense_gazebo_plugin)/urdf/d435.urdf.xacro"/>
+    <xacro:sensor_d435 parent="pole">
+        <origin xyz="0 0 1.5" rpy="0 0 0"/>
+    </xacro:sensor_d435>
 <!-- IMU DEFINITION -->
     <link name="imu_link">

File: couchmobile_description/urdf/realsense-d435.macro.xacro (robot description, xacro)
@@ -127,9 +127,4 @@
 <!-- **********************************************************-->
 <!-- GAZEBO DEFINITIONS ***************************************-->
-    <!-- Load plugin to the model ("robot" in urdf format)-->
-    <gazebo>
-        <plugin name="${prefix}d435" filename="librealsense_gazebo_plugin.so"/>
-        <!--<pose frame="">0 0 0.015 0 0 0</pose>-->
-    </gazebo>
     <!-- Load parameters to model's main link-->
     <gazebo reference="camera_link">
@@ -239,4 +234,28 @@
         </sensor>
     </gazebo>
+<!-- Load plugin to the model ("robot" in urdf format)-->
+    <gazebo>
+        <plugin name="${prefix}d435" filename="librealsense_gazebo_plugin.so"/>
+        <depthUpdateRate>60.0</depthUpdateRate>
+      	<colorUpdateRate>60.0</colorUpdateRate>
+      	<infraredUpdateRate>60.0</infraredUpdateRate>
+      	<depthTopicName>depth/image_raw</depthTopicName>
+      	<depthCameraInfoTopicName>depth/camera_info</depthCameraInfoTopicName>
+      	<colorTopicName>color/image_raw</colorTopicName>
+      	<colorCameraInfoTopicName>color/camera_info</colorCameraInfoTopicName>
+      	<infrared1TopicName>infra1/image_raw</infrared1TopicName>
+      	<infrared1CameraInfoTopicName>infra1/camera_info</infrared1CameraInfoTopicName>
+      	<infrared2TopicName>infra2/image_raw</infrared2TopicName>
+      	<infrared2CameraInfoTopicName>infra2/camera_info</infrared2CameraInfoTopicName>
+      	<colorOpticalframeName>camera_color_optical_frame</colorOpticalframeName>
+      	<depthOpticalframeName>camera_depth_optical_frame</depthOpticalframeName>
+      	<infrared1OpticalframeName>camera_right_ir_optical_frame</infrared1OpticalframeName>
+      	<infrared2OpticalframeName>camera_left_ir_optical_frame</infrared2OpticalframeName>
+      	<rangeMinDepth>0.2</rangeMinDepth>
+      	<rangeMaxDepth>10.0</rangeMaxDepth>
+      	<pointCloud>false</pointCloud>
+      	<pointCloudTopicName>depth/points</pointCloudTopicName>
+      	<pointCloudCutoff>0.5</pointCloudCutoff>
+    </gazebo>
 </xacro:macro>
 </robot>
